File: PCBv2/walle.sch (KiCad schematic (older format))
At the start: 30 parts, among them IC1 L293D, J1 Conn_01x07, J10 Head_Motor_B, J11 Head_Motor_A, J2 Front_LED, J3 Track_Motor_A, J4 5V, J5 Speaker, J6 GND, J7 Conn_01x08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

Commit message: assigned footprints
Parts:
- D1, D2, D3, D4, D5, D6, D7, D8: footprint (none) -> Diodes_THT:D_5KP_P7.62mm_Vertical_AnodeUp
- J1: footprint (none) -> Pin_Headers:Pin_Header_Straight_1x07_Pitch2.54mm
- J10, J11, J8: footprint (none) -> Pin_Headers:Pin_Header_Straight_1x02_Pitch2.54mm_SMD_Pin1Left
- J7: footprint (none) -> Pin_Headers:Pin_Header_Straight_1x08_Pitch2.54mm
Changed lines of the file:
@@
 F 0 "D2" H 1150 4600 50  0000 C CNN
 F 1 "D" H 1150 4400 50  0000 C CNN
-F 2 "" H 1150 4500 50  0001 C CNN
+F 2 "Diodes_THT:D_5KP_P7.62mm_Vertical_AnodeUp" H 1150 4500 50  0001 C CNN
 F 3 "" H 1150 4500 50  0001 C CNN
 	1    1150 4500
@@
 F 0 "D1" H 1150 4300 50  0000 C CNN
 F 1 "D" H 1150 4100 50  0000 C CNN
-F 2 "" H 1150 4200 50  0001 C CNN
+F 2 "Diodes_THT:D_5KP_P7.62mm_Vertical_AnodeUp" H 1150 4200 50  0001 C CNN
 F 3 "" H 1150 4200 50  0001 C CNN
 	1    1150 4200
@@
 F 0 "J8" H 1200 5050 50  0000 C CNN
 F 1 "Track_Motor_B" V 1300 5000 50  0000 C CNN
-F 2 "" H 1200 4950 50  0001 C CNN
+F 2 "Pin_Headers:Pin_Header_Straight_1x02_Pitch2.54mm_SMD_Pin1Left" H 1200 4950 50  0001 C CNN
 F 3 "" H 1200 4950 50  0001 C CNN
 	1    1200 4950
@@
 F 0 "D3" H 1400 4900 50  0000 C CNN
 F 1 "D" H 1400 4700 50  0000 C CNN
-F 2 "" H 1400 4800 50  0001 C CNN
+F 2 "Diodes_THT:D_5KP_P7.62mm_Vertical_AnodeUp" H 1400 4800 50  0001 C CNN
 F 3 "" H 1400 4800 50  0001 C CNN
 	1    1400 4800
@@
 F 0 "D4" H 1400 5200 50  0000 C CNN
 F 1 "D" H 1400 5000 50  0000 C CNN
-F 2 "" H 1400 5100 50  0001 C CNN
+F 2 "Diodes_THT:D_5KP_P7.62mm_Vertical_AnodeUp" H 1400 5100 50  0001 C CNN
 F 3 "" H 1400 5100 50  0001 C CNN
 	1    1400 5100
@@
 F 0 "J11" H 4200 4450 50  0000 C CNN
 F 1 "Head_Motor_A" V 4300 4350 50  0000 C CNN
-F 2 "" H 4200 4350 50  0001 C CNN
+F 2 "Pin_Headers:Pin_Header_Straight_1x02_Pitch2.54mm_SMD_Pin1Left" H 4200 4350 50  0001 C CNN
 F 3 "" H 4200 4350 50  0001 C CNN
 	1    4200 4350
@@
 F 0 "D8" H 4000 4600 50  0000 C CNN
 F 1 "D" H 4000 4400 50  0000 C CNN
-F 2 "" H 4000 4500 50  0001 C CNN
+F 2 "Diodes_THT:D_5KP_P7.62mm_Vertical_AnodeUp" H 4000 4500 50  0001 C CNN
 F 3 "" H 4000 4500 50  0001 C CNN
 	1    4000 4500
@@
 F 0 "D7" H 4000 4300 50  0000 C CNN
 F 1 "D" H 4000 4100 50  0000 C CNN
-F 2 "" H 4000 4200 50  0001 C CNN
+F 2 "Diodes_THT:D_5KP_P7.62mm_Vertical_AnodeUp" H 4000 4200 50  0001 C CNN
 F 3 "" H 4000 4200 50  0001 C CNN
 	1    4000 4200
@@
 F 0 "J10" H 3600 5050 50  0000 C CNN
 F 1 "Head_Motor_B" V 3700 4950 50  0000 C CNN
-F 2 "" H 3600 4950 50  0001 C CNN
+F 2 "Pin_Headers:Pin_Header_Straight_1x02_Pitch2.54mm_SMD_Pin1Left" H 3600 4950 50  0001 C CNN
 F 3 "" H 3600 4950 50  0001 C CNN
 	1    3600 4950
@@
 F 0 "D6" H 3400 5200 50  0000 C CNN
 F 1 "D" H 3400 5000 50  0000 C CNN
-F 2 "" H 3400 5100 50  0001 C CNN
+F 2 "Diodes_THT:D_5KP_P7.62mm_Vertical_AnodeUp" H 3400 5100 50  0001 C CNN
 F 3 "" H 3400 5100 50  0001 C CNN
 	1    3400 5100
@@
 F 0 "D5" H 3400 4900 50  0000 C CNN
 F 1 "D" H 3400 4700 50  0000 C CNN
-F 2 "" H 3400 4800 50  0001 C CNN
+F 2 "Diodes_THT:D_5KP_P7.62mm_Vertical_AnodeUp" H 3400 4800 50  0001 C CNN
 F 3 "" H 3400 4800 50  0001 C CNN
 	1    3400 4800
@@
 F 0 "J7" H 7400 1850 50  0000 C CNN
 F 1 "Conn_01x08" H 7400 950 50  0000 C CNN
-F 2 "" H 7400 1450 50  0001 C CNN
+F 2 "Pin_Headers:Pin_Header_Straight_1x08_Pitch2.54mm" H 7400 1450 50  0001 C CNN
 F 3 "" H 7400 1450 50  0001 C CNN
 	1    7400 1450
@@
 F 0 "J1" H 2700 2150 50  0000 C CNN
 F 1 "Conn_01x07" H 2700 1350 50  0000 C CNN
-F 2 "" H 2700 1750 50  0001 C CNN
+F 2 "Pin_Headers:Pin_Header_Straight_1x07_Pitch2.54mm" H 2700 1750 50  0001 C CNN
 F 3 "" H 2700 1750 50  0001 C CNN
 	1    2700 1750
@@
 $EndComp
 $Comp
-L VCC #PWR?
+L VCC #PWR033
 U 1 1 59DCF3EB
 P 4000 4050
-F 0 "#PWR?" H 4000 3900 50  0001 C CNN
+F 0 "#PWR033" H 4000 3900 50  0001 C CNN
 F 1 "VCC" H 4000 4200 50  0000 C CNN
 F 2 "" H 4000 4050 50  0001 C CNN
@@
 $EndComp
 $Comp
-L VCC #PWR?
+L VCC #PWR034
 U 1 1 59DCF43B
 P 3400 4650
-F 0 "#PWR?" H 3400 4500 50  0001 C CNN
+F 0 "#PWR034" H 3400 4500 50  0001 C CNN
 F 1 "VCC" H 3400 4800 50  0000 C CNN
 F 2 "" H 3400 4650 50  0001 C CNN
@@
 $EndComp
 $Comp
-L VCC #PWR?
+L VCC #PWR035
 U 1 1 59DCF48B
 P 1150 4050
-F 0 "#PWR?" H 1150 3900 50  0001 C CNN
+F 0 "#PWR035" H 1150 3900 50  0001 C CNN
 F 1 "VCC" H 1150 4200 50  0000 C CNN
 F 2 "" H 1150 4050 50  0001 C CNN
@@
 $EndComp
 $Comp
-L VCC #PWR?
+L VCC #PWR036
 U 1 1 59DCF4DB
 P 1400 4650
-F 0 "#PWR?" H 1400 4500 50  0001 C CNN
+F 0 "#PWR036" H 1400 4500 50  0001 C CNN
 F 1 "VCC" H 1400 4800 50  0000 C CNN
 F 2 "" H 1400 4650 50  0001 C CNN

Commit message: ratsnest
Parts:
- D1, D2, D3, D4, D5, D6, D7, D8: footprint Diodes_THT:D_5KP_P7.62mm_Vertical_AnodeUp -> Diodes_THT:D_A-405_P2.54mm_Vertical_AnodeUp
- J10, J11, J8: footprint Pin_Headers:Pin_Header_Straight_1x02_Pitch2.54mm_SMD_Pin1Left -> Pin_Headers:Pin_Header_Straight_1x01_Pitch2.54mm
- J3, J5, J9: footprint Pin_Headers:Pin_Header_Straight_1x01_Pitch2.54mm_SMD_Pin1Left -> Pin_Headers:Pin_Header_Straight_1x01_Pitch2.54mm
- R1, R2, R3, R4, R5, R6, R7: footprint Discret:R1 -> Resistors_THT:R_Axial_DIN0204_L3.6mm_D1.6mm_P1.90mm_Vertical
Changed lines of the file:
@@
 F 0 "R1" V 3780 3150 50  0000 C CNN
 F 1 "3k" V 3700 3150 50  0000 C CNN
-F 2 "Discret:R1" V 3630 3150 50  0001 C CNN
+F 2 "Resistors_THT:R_Axial_DIN0204_L3.6mm_D1.6mm_P1.90mm_Vertical" V 3630 3150 50  0001 C CNN
 F 3 "" H 3700 3150 50  0001 C CNN
 	1    3700 3150
@@
 F 0 "J3" H 950 4450 50  0000 C CNN
 F 1 "Track_Motor_A" V 1050 4350 50  0000 C CNN
-F 2 "Pin_Headers:Pin_Header_Straight_1x01_Pitch2.54mm_SMD_Pin1Left" H 950 4350 50  0001 C CNN
+F 2 "Pin_Headers:Pin_Header_Straight_1x01_Pitch2.54mm" H 950 4350 50  0001 C CNN
 F 3 "" H 950 4350 50  0001 C CNN
 	1    950  4350
@@
 F 0 "R3" V 6880 2550 50  0000 C CNN
 F 1 "2k2" V 6800 2550 50  0000 C CNN
-F 2 "Discret:R1" V 6730 2550 50  0001 C CNN
+F 2 "Resistors_THT:R_Axial_DIN0204_L3.6mm_D1.6mm_P1.90mm_Vertical" V 6730 2550 50  0001 C CNN
 F 3 "" H 6800 2550 50  0001 C CNN
 	1    6800 2550
@@
 F 0 "R2" V 6680 2700 50  0000 C CNN
 F 1 "3k3" V 6600 2700 50  0000 C CNN
-F 2 "Discret:R1" V 6530 2700 50  0001 C CNN
+F 2 "Resistors_THT:R_Axial_DIN0204_L3.6mm_D1.6mm_P1.90mm_Vertical" V 6530 2700 50  0001 C CNN
 F 3 "" H 6600 2700 50  0001 C CNN
 	1    6600 2700
@@
 F 0 "J5" H 3250 2050 50  0000 C CNN
 F 1 "Speaker" V 3350 1950 50  0000 C CNN
-F 2 "Pin_Headers:Pin_Header_Straight_1x01_Pitch2.54mm_SMD_Pin1Left" H 3250 1950 50  0001 C CNN
+F 2 "Pin_Headers:Pin_Header_Straight_1x01_Pitch2.54mm" H 3250 1950 50  0001 C CNN
 F 3 "" H 3250 1950 50  0001 C CNN
 	1    3250 1950
@@
 F 0 "R7" V 6730 2100 50  0000 C CNN
 F 1 "2k2" V 6650 2100 50  0000 C CNN
-F 2 "Discret:R1" V 6580 2100 50  0001 C CNN
+F 2 "Resistors_THT:R_Axial_DIN0204_L3.6mm_D1.6mm_P1.90mm_Vertical" V 6580 2100 50  0001 C CNN
 F 3 "" H 6650 2100 50  0001 C CNN
 	1    6650 2100
@@
 F 0 "R6" V 6580 2250 50  0000 C CNN
 F 1 "3k3" V 6500 2250 50  0000 C CNN
-F 2 "Discret:R1" V 6430 2250 50  0001 C CNN
+F 2 "Resistors_THT:R_Axial_DIN0204_L3.6mm_D1.6mm_P1.90mm_Vertical" V 6430 2250 50  0001 C CNN
 F 3 "" H 6500 2250 50  0001 C CNN
 	1    6500 2250
@@
 F 0 "R4" V 3580 2050 50  0000 C CNN
 F 1 "2k2" V 3500 2050 50  0000 C CNN
-F 2 "Discret:R1" V 3430 2050 50  0001 C CNN
+F 2 "Resistors_THT:R_Axial_DIN0204_L3.6mm_D1.6mm_P1.90mm_Vertical" V 3430 2050 50  0001 C CNN
 F 3 "" H 3500 2050 50  0001 C CNN
 	1    3500 2050
@@
 F 0 "R5" V 3730 2200 50  0000 C CNN
 F 1 "3k3" V 3650 2200 50  0000 C CNN
-F 2 "Discret:R1" V 3580 2200 50  0001 C CNN
+F 2 "Resistors_THT:R_Axial_DIN0204_L3.6mm_D1.6mm_P1.90mm_Vertical" V 3580 2200 50  0001 C CNN
 F 3 "" H 3650 2200 50  0001 C CNN
 	1    3650 2200
@@
 F 0 "J9" H 8600 2800 50  0000 C CNN
 F 1 "SPKR_GND" V 8700 2700 50  0000 C CNN
-F 2 "Pin_Headers:Pin_Header_Straight_1x01_Pitch2.54mm_SMD_Pin1Left" H 8600 2700 50  0001 C CNN
+F 2 "Pin_Headers:Pin_Header_Straight_1x01_Pitch2.54mm" H 8600 2700 50  0001 C CNN
 F 3 "" H 8600 2700 50  0001 C CNN
 	1    8600 2700
@@
 F 0 "D2" H 1150 4600 50  0000 C CNN
 F 1 "D" H 1150 4400 50  0000 C CNN
-F 2 "Diodes_THT:D_5KP_P7.62mm_Vertical_AnodeUp" H 1150 4500 50  0001 C CNN
+F 2 "Diodes_THT:D_A-405_P2.54mm_Vertical_AnodeUp" H 1150 4500 50  0001 C CNN
 F 3 "" H 1150 4500 50  0001 C CNN
 	1    1150 4500
@@
 F 0 "D1" H 1150 4300 50  0000 C CNN
 F 1 "D" H 1150 4100 50  0000 C CNN
-F 2 "Diodes_THT:D_5KP_P7.62mm_Vertical_AnodeUp" H 1150 4200 50  0001 C CNN
+F 2 "Diodes_THT:D_A-405_P2.54mm_Vertical_AnodeUp" H 1150 4200 50  0001 C CNN
 F 3 "" H 1150 4200 50  0001 C CNN
 	1    1150 4200
@@
 F 0 "J8" H 1200 5050 50  0000 C CNN
 F 1 "Track_Motor_B" V 1300 5000 50  0000 C CNN
-F 2 "Pin_Headers:Pin_Header_Straight_1x02_Pitch2.54mm_SMD_Pin1Left" H 1200 4950 50  0001 C CNN
+F 2 "Pin_Headers:Pin_Header_Straight_1x01_Pitch2.54mm" H 1200 4950 50  0001 C CNN
 F 3 "" H 1200 4950 50  0001 C CNN
 	1    1200 4950
@@
 F 0 "D3" H 1400 4900 50  0000 C CNN
 F 1 "D" H 1400 4700 50  0000 C CNN
-F 2 "Diodes_THT:D_5KP_P7.62mm_Vertical_AnodeUp" H 1400 4800 50  0001 C CNN
+F 2 "Diodes_THT:D_A-405_P2.54mm_Vertical_AnodeUp" H 1400 4800 50  0001 C CNN
 F 3 "" H 1400 4800 50  0001 C CNN
 	1    1400 4800
@@
 F 0 "D4" H 1400 5200 50  0000 C CNN
 F 1 "D" H 1400 5000 50  0000 C CNN
-F 2 "Diodes_THT:D_5KP_P7.62mm_Vertical_AnodeUp" H 1400 5100 50  0001 C CNN
+F 2 "Diodes_THT:D_A-405_P2.54mm_Vertical_AnodeUp" H 1400 5100 50  0001 C CNN
 F 3 "" H 1400 5100 50  0001 C CNN
 	1    1400 5100
@@
 F 0 "J11" H 4200 4450 50  0000 C CNN
 F 1 "Head_Motor_A" V 4300 4350 50  0000 C CNN
-F 2 "Pin_Headers:Pin_Header_Straight_1x02_Pitch2.54mm_SMD_Pin1Left" H 4200 4350 50  0001 C CNN
+F 2 "Pin_Headers:Pin_Header_Straight_1x01_Pitch2.54mm" H 4200 4350 50  0001 C CNN
 F 3 "" H 4200 4350 50  0001 C CNN
 	1    4200 4350
@@
 F 0 "D8" H 4000 4600 50  0000 C CNN
 F 1 "D" H 4000 4400 50  0000 C CNN
-F 2 "Diodes_THT:D_5KP_P7.62mm_Vertical_AnodeUp" H 4000 4500 50  0001 C CNN
+F 2 "Diodes_THT:D_A-405_P2.54mm_Vertical_AnodeUp" H 4000 4500 50  0001 C CNN
 F 3 "" H 4000 4500 50  0001 C CNN
 	1    4000 4500
@@
 F 0 "D7" H 4000 4300 50  0000 C CNN
 F 1 "D" H 4000 4100 50  0000 C CNN
-F 2 "Diodes_THT:D_5KP_P7.62mm_Vertical_AnodeUp" H 4000 4200 50  0001 C CNN
+F 2 "Diodes_THT:D_A-405_P2.54mm_Vertical_AnodeUp" H 4000 4200 50  0001 C CNN
 F 3 "" H 4000 4200 50  0001 C CNN
 	1    4000 4200
@@
 F 0 "J10" H 3600 5050 50  0000 C CNN
 F 1 "Head_Motor_B" V 3700 4950 50  0000 C CNN
-F 2 "Pin_Headers:Pin_Header_Straight_1x02_Pitch2.54mm_SMD_Pin1Left" H 3600 4950 50  0001 C CNN
+F 2 "Pin_Headers:Pin_Header_Straight_1x01_Pitch2.54mm" H 3600 4950 50  0001 C CNN
 F 3 "" H 3600 4950 50  0001 C CNN
 	1    3600 4950
@@
 F 0 "D6" H 3400 5200 50  0000 C CNN
 F 1 "D" H 3400 5000 50  0000 C CNN
-F 2 "Diodes_THT:D_5KP_P7.62mm_Vertical_AnodeUp" H 3400 5100 50  0001 C CNN
+F 2 "Diodes_THT:D_A-405_P2.54mm_Vertical_AnodeUp" H 3400 5100 50  0001 C CNN
 F 3 "" H 3400 5100 50  0001 C CNN
 	1    3400 5100
@@
 F 0 "D5" H 3400 4900 50  0000 C CNN
 F 1 "D" H 3400 4700 50  0000 C CNN
-F 2 "Diodes_THT:D_5KP_P7.62mm_Vertical_AnodeUp" H 3400 4800 50  0001 C CNN
+F 2 "Diodes_THT:D_A-405_P2.54mm_Vertical_AnodeUp" H 3400 4800 50  0001 C CNN
 F 3 "" H 3400 4800 50  0001 C CNN
 	1    3400 4800
