File: PCBv2/walle.kicad_pcb (KiCad board)
At the start: 2 copper layers, 30 parts, among them IC1 L293D, J1 Conn_01x07, J10 Head_Motor_B, J11 Head_Motor_A, J2 Front_LED, J3 Track_Motor_A, J4 5V, J5 Speaker, J6 GND, J7 Conn_01x08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

Commit message: final PCB
Parts:
- added G***: LOGO, OPENHARDWARE:OSHWLOGO0.75IN, F.Cu at (161.5, 58.0)
- added REF**: SolderWirePad_single_1-2mmDrill, Wire_Pads:SolderWirePad_single_1-2mmDrill, F.Cu at (119.6, 85.1)
- added REF**: SolderWirePad_single_1-2mmDrill, Wire_Pads:SolderWirePad_single_1-2mmDrill, F.Cu at (121.4, 110.5)
- added REF**: SolderWirePad_single_1-2mmDrill, Wire_Pads:SolderWirePad_single_1-2mmDrill, F.Cu at (145.0, 106.2)
- added REF**: SolderWirePad_single_1-2mmDrill, Wire_Pads:SolderWirePad_single_1-2mmDrill, F.Cu at (152.4, 138.2)
- J10: value Head_Motor_B -> <HD_MTR_B
- J3: value Track_Motor_A -> TR_MTR_A
- J5: value Speaker -> SPKR
- J8: value Track_Motor_B -> TRK_MTR_B
- moved D2 119.0 mm to (101.1, 111.6)
- moved D7 115.6 mm to (105.0, 66.5), turned to 180 degrees
- moved D1 114.7 mm to (101.1, 105.2), turned to 270 degrees
- moved D8 113.0 mm to (110.9, 66.9), turned to 270 degrees
- moved D6 112.8 mm to (110.5, 76.1)
- moved D5 110.0 mm to (105.3, 73.5), turned to 270 degrees
- moved D3 108.8 mm to (105.9, 105.2)
- moved D4 98.1 mm to (113.8, 105.2)
- moved R7 94.3 mm to (148.3, 73.7), turned to 270 degrees
- moved J11 92.9 mm to (108.7, 62.2)
- moved U2 91.0 mm to (128.4, 79.2), turned to 180 degrees
- moved SW1 88.8 mm to (130.9, 70.4)
- moved R6 88.6 mm to (148.3, 78.2), turned to 180 degrees
- moved R3 83.1 mm to (151.3, 73.7), turned to 270 degrees
- moved J10 80.7 mm to (100.6, 76.1)
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Routing:
- net VCC: track 0.00 -> 104.4 mm, vias 0 -> 3
- net /5V_Regulated: track 0.00 -> 91.9 mm, vias 0 -> 1
- net /USB_D-: track 0.00 -> 62.4 mm, vias 0 -> 2
- net /USB_D+: track 0.00 -> 57.3 mm, vias 0 -> 2
- net /H_top_A: track 0.00 -> 56.0 mm
- net /H_top_EN: track 0.00 -> 53.1 mm, vias 0 -> 1
- net Net-(D7-Pad2): track 0.00 -> 49.7 mm
- net Net-(J1-Pad1): track 0.00 -> 47.7 mm
- net /H_top_2A: track 0.00 -> 47.6 mm, vias 0 -> 1
- net /H_1A: track 0.00 -> 44.1 mm, vias 0 -> 1
- net /H_EN: track 0.00 -> 39.5 mm
- net GND: track 0.00 -> 38.9 mm, vias 0 -> 3
- net /H_2A: track 0.00 -> 37.5 mm
- net Net-(D3-Pad2): track 0.00 -> 33.2 mm
- net Net-(D1-Pad2): track 0.00 -> 30.3 mm
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- added copper zone on B.Cu, net GND
- added copper zone on F.Cu, net GND
Other:
- board outline added: 82.4 x 57.9 mm
- net class Default: trace_width 0.25 -> 0.6; via_dia 0.6 -> 0.66; via_drill 0.4 -> 0.34
- net class Power added: clearance 0.4, trace_width 1.2, via_dia 1, via_drill 0.5
- board text added: "Wallsy Main Board © Stef Pletinck github.com/Epse/Wallsy"
